File: EagleFiles/board.brd (EAGLE design)
At the start: 45 parts

Commit message: first ideas of board, some data sheets, firt schematic test
Parts:
- added E$46, E$47, E$48: (no value), linear-technology:TSOT23-6
Changed lines of the file:
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@@
 <layer number="97" name="Info" color="7" fill="1" visible="no" active="no"/>
 <layer number="98" name="Guide" color="6" fill="1" visible="no" active="no"/>
+<layer number="99" name="SpiceOrder" color="5" fill="1" visible="no" active="no"/>
 <layer number="100" name="Muster" color="7" fill="1" visible="no" active="no"/>
 <layer number="101" name="Patch_Top" color="12" fill="4" visible="yes" active="yes"/>
@@
 <element name="E$23" library="div" package="USB-B-SMD" value="" x="31.75" y="17.78" rot="MR90"/>
 <element name="E$45" library="analog-devices" package="SO14" value="" x="30.48" y="72.39" rot="MR0"/>
+<element name="E$46" library="linear-technology" package="TSOT23-6" value="" x="63.5" y="45.72" rot="MR0"/>
+<element name="E$47" library="linear-technology" package="TSOT23-6" value="" x="68.58" y="40.64" rot="MR90"/>
+<element name="E$48" library="linear-technology" package="TSOT23-6" value="" x="68.58" y="34.29" rot="MR90"/>
 </elements>
 <signals>
