File: EagleFiles/ledboard_RC1/REV1.sch (EAGLE design)
At the start: 164 parts, among them K1 694106105102, Q1_24MHZ ECS-240-18-23A-EN-TR, X1 USBSMD

Commit message: updated board
Parts:
- added C79: 100NF, rcl:C-EUC0603
- LDO: value TPS79933 -> TPS73633; device TPS79933:TPS79933 -> TPS73633:TPS73633
Connections:
- net +5V: now also C79.1
- net GND: now also C79.2
Other:
- note added: "100n gehört zum WE-TVS"
- note added: "ToDo... - Kondensatoren/Spulen zur Spannungsglättung einfügen"
- note removed: "ToDo... - Kondensatoren/Spulen zur Spannungsglättung einfügen - Kondensator beim LDO Eingang"
- moved on the sheet: LDO

Commit message: First layout done, few changes for easier routing
Parts:
- removed R10: 47, rcl:R-EU_R0603
- C67: value 4.7mu -> 4.7µF
- C79: value 100NF -> 100nF
- JP1: device pinhead:PINHD-2X10 -> pinhead:PINHD-2X10_2.54-SMD
- T1, T2: value (none) -> SI4465DY
- renumbered SI4465DY_1 to T1, SI4465DY_2 to T2
Connections:
- net N$47 renamed D+_TMP
- net N$64 renamed D-_TMP
- removed net N$52: LED35.DO, LED36.DI
- removed net VREF+: MCU.VREF+, R10.2
- new net N$47: LED36.DI, R1.2
- net +3V3: now also MCU.VREF+; no longer R10.1
- net D+: now also C69.2, R5.2; no longer C70.2, R4.2, R6.1
- net D-: now also C70.2, R4.2, R6.1; no longer C69.2, R5.2
- net DATA_IN_1_HIGH: now also R3.1; no longer R1.1
- net DATA_IN_2_HIGH: now also R1.1; no longer R3.1
- net N$1: now also LED45.DO; no longer R1.2
- net N$22: now also R3.2; no longer LED5.DO
- net N$32: now also LED15.DO; no longer R3.2
- net N$65: now also L1.3; no longer L1.2
- net N$66: now also L1.2; no longer L1.3
Other:
- note added: "ToDo... - Kondensatoren/Spulen zur Spannungsglättung einfügen - LTC4412: 100nF zwischen Vin and GND"
- note removed: "ToDo... - Kondensatoren/Spulen zur Spannungsglättung einfügen"
- moved on the sheet: L1, R1, R3

Commit message: update
Parts:
- removed FERRITBEAD: MLS0805-4S7-102, MLS0805:MLS0805-4S7-102
- added C80: 100nF, rcl:C-EUC0603
Connections:
- removed net N$54: LED37.DO, LED38.DI
- removed net N$62: C66.1, FERRITBEAD.1, LDO.OUT
- removed net N$70: 0.5.O, T1.D
- new net N$52: LED35.DO, LED36.DI
- new net VBUS_S: 0.5.O, C68.2, D1.VDD, T1.D
- net +3V3: now also C66.1, LDO.OUT; no longer FERRITBEAD.2
- net D+: now also R6.1
- net D-: no longer R6.1
- net DATA_IN_1_HIGH: now also R1.1; no longer R3.1
- net DATA_IN_2_HIGH: now also R3.1; no longer R1.1
- net GND: now also C80.2
- net N$22: now also LED7.DI; no longer LED6.DI
- net N$23: now also LED5.DO, LED6.DI; no longer LED6.DO, LED7.DI
- net N$47: now also LED38.DI; no longer LED36.DI
- net VBUS: no longer C68.2, D1.VDD
- net V_5: now also C80.1
Other:
- moved on the sheet: 4, C68
