File: Eagle/ledboard_RC1/REV1.brd (EAGLE design)
At the start: 100 x 100 mm, 166 parts, among them K1 694106105102, Q1_24MHZ ECS-240-18-23A-EN-TR, T1 SI4465DY, T2 SI4465DY, X1 USBSMD, X2 RJHSE5380

Commit message: updated board layout
Parts:
- moved R1 3.41 mm to (80.6, 61.2), flipped to the bottom, turned to 180 degrees
- moved R3 1.84 mm to (81.3, 65.7), flipped to the bottom, turned to 180 degrees
- moved C30 0.16 mm to (35.6, 94.8), flipped to the top, turned to 108 degrees
- moved C17 0.16 mm to (45.2, 3.33), flipped to the top, turned to 264 degrees
- moved C12 0.16 mm to (88.2, 22.4), flipped to the top, turned to 324 degrees
- moved C14 0.16 mm to (73.6, 9.37), flipped to the top, turned to 300 degrees
- moved C16 0.16 mm to (55.0, 3.33), flipped to the top, turned to 276 degrees
- moved C19 0.16 mm to (26.6, 9.37), flipped to the top, turned to 240 degrees
- moved C8 0.16 mm to (96.1, 59.8), flipped to the top, turned to 12 degrees
- moved C5 0.16 mm to (81.6, 85.0), flipped to the top, turned to 48 degrees
- moved C13 0.16 mm to (81.6, 15.1), flipped to the top, turned to 312 degrees
- moved C25 0.16 mm to (4.16, 59.8), turned to 168 degrees
- moved C26 0.16 mm to (7.19, 69.2), flipped to the top, turned to 156 degrees
- moved C6 0.16 mm to (88.2, 77.7), flipped to the top, turned to 36 degrees
- moved C22 0.16 mm to (7.19, 31.0), flipped to the top, turned to 204 degrees
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Routing:
- net N$47: track 3.46 -> 0.00 mm
- net +3V3: track 160.0 -> 162.0 mm
